File: anise60bnav/kbd-gen.kicad_pcb (KiCad board)
At the start: 2 copper layers, 284.6 x 94.2 mm, 146 parts, among them CN1 BTB, CN2 BTB, P1 P, P2 P

Commit message: add more layout
Routing:
- net c3: track 139.3 -> 138.2 mm
- net c7: track 257.4 -> 256.5 mm

Commit message: update with anise90 seris/ outline and holes are not fully ready
Routing:
- net VCC: track 1666.8 -> 1659.4 mm
- net c2: track 141.7 -> 140.1 mm
- net GND: track 1609.6 -> 1609.0 mm
