File: anise60b/kbd-gen.kicad_pcb (KiCad board)
At the start: 2 copper layers, 284.6 x 94.2 mm, 148 parts, among them CN1 BTB, CN2 BTB

Commit message: add more layout
Parts:
- added P1: P, Connector_PinHeader_2.00mm:PinHeader_1x04_P2.00mm_Vertical, B.Cu at (65.2, 109.9)
- added P2: P, Connector_PinHeader_2.00mm:PinHeader_1x04_P2.00mm_Vertical, B.Cu at (344.4, 115.9)
Connections:
- net S17_16 renamed S17_18
- net led2_17 renamed led1_17
- CN1 pad 33: VCC -> (no net)
- CN1 pad 34: GND -> (no net)
- CN1 pad 4: (no net) -> sdaL
- CN1 pad 6: (no net) -> sclL
- CN2 pad 33: VCC -> (no net)
- CN2 pad 34: GND -> (no net)
- CN2 pad 4: (no net) -> sdaR
- CN2 pad 6: (no net) -> sclR
Routing:
- net sclR: track 0.00 -> 127.7 mm, vias 0 -> 1
- net sdaR: track 0.00 -> 123.7 mm, vias 0 -> 1
- net sclL: track 0.00 -> 106.9 mm, vias 0 -> 2
- net sdaL: track 0.00 -> 104.9 mm, vias 0 -> 2
- net VCC: track 1707.8 -> 1750.2 mm
- net GND: track 1712.7 -> 1741.1 mm
- net r2: track 319.7 -> 326.5 mm
Other:
- board text added: "G V C D"

Commit message: update for 24 Feb 2023 release
Routing:
- net (no net): track 45.3 -> 0.00 mm
Changed lines of the file:
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@@
     (pad_to_mask_clearance 0)
     (aux_axis_origin 62.49 159.02)
+    (grid_origin 182.11 71.88)
     (pcbplotparams
       (layerselection 0x00010fc_ffffffff)
@@
     (effects (font (size 1 1) (thickness 0.2)) (justify left))
   )
-  (segment (start 182.127889 71.919749) (end 182.170638 71.877) (width 0.25) (layer "F.Cu") (net 0))
-  (segment (start 137.955251 71.919749) (end 182.127889 71.919749) (width 0.25) (layer "F.Cu") (net 0))
-  (segment (start 137.2 72.675) (end 137.955251 71.919749) (width 0.25) (layer "F.Cu") (net 0))
   (segment (start 201.365751 75.340751) (end 193.659249 75.340751) (width 0.2) (layer "F.Cu") (net 1))
   (segment (start 183.7 75.325) (end 180.338391 75.325) (width 0.2) (layer "F.Cu") (net 1))
