File: anise90a/kbd-gen.kicad_pcb (KiCad board)
At the start: 2 copper layers, 332.2 x 119.4 mm, 189 parts, among them CN1 BTB, CN2 BTB, P1 P, P2 P

Commit message: update for 24 Feb 2023 release
Parts:
- removed the REF** at (359.4, 59.0)
- removed the REF** at (45.1, 59.0)
- added ?: , , F.Cu at (186.6, 63.0)
- added ?: , , F.Cu at (175.3, 63.0)
- added ?: , , F.Cu at (175.1, 60.8)
- added ?: , , F.Cu at (205.7, 63.0)
- added ?: , , F.Cu at (194.3, 60.9)
- added ?: , , F.Cu at (183.7, 59.9)
- added ?: , , F.Cu at (204.8, 58.4)
- added ?: , , F.Cu at (197.2, 63.9)
- added ?: , , F.Cu at (202.8, 59.9)
- added ?: , , F.Cu at (178.2, 63.9)
- added ?: , , F.Cu at (194.4, 63.0)
- added ?: , , F.Cu at (200.0, 62.0)
- added ?: , , F.Cu at (180.9, 61.9)
- added ?: , , F.Cu at (185.7, 58.1)
- added REF**: PinHeader_1x03_P1.27mm_Vertical, Connector_PinHeader_1.27mm:PinHeader_1x03_P1.27mm_Vertical, B.Cu at (354.4, 53.0)
- added REF**: PinHeader_1x03_P1.27mm_Vertical, Connector_PinHeader_1.27mm:PinHeader_1x03_P1.27mm_Vertical, B.Cu at (40.1, 53.0)
- added REF**: PinHeader_1x03_P1.27mm_Vertical, Connector_PinHeader_1.27mm:PinHeader_1x03_P1.27mm_Vertical, B.Cu at (369.4, 53.0)
- added REF**: PinHeader_1x03_P1.27mm_Vertical, Connector_PinHeader_1.27mm:PinHeader_1x03_P1.27mm_Vertical, B.Cu at (55.1, 53.0)
- added S12: MX_LED, Keyboard:MXHS-1U-RGB-ALI-3528-HOLE-NOPAD, F.Cu at (95.2, 50.0)
- moved S16 19.1 mm to (176.2, 50.0)
- moved S110 14.3 mm to (257.2, 50.0)
- moved CN1 14.3 mm to (142.9, 59.4)
- moved S13 14.3 mm to (114.3, 50.0)
- moved S14 14.3 mm to (133.3, 50.0)
- moved S15 14.3 mm to (152.4, 50.0)
- moved ? 9.53 mm to (206.4, 40.8)
- moved ? 9.53 mm to (185.5, 43.5)
- moved ? 9.53 mm to (187.4, 40.8)
- moved ? 9.53 mm to (223.8, 50.0)
- moved ? 9.53 mm to (185.7, 50.0)
- moved ? 9.53 mm to (204.5, 43.5)
- moved ? 9.53 mm to (204.8, 50.0)
- moved ? 9.53 mm to (203.1, 40.8)
- moved S18 9.53 mm to (214.3, 50.0)
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Connections:
- net S16_17 renamed S18_17
- net S27_28 renamed S27_26
- S11 pad DO: S11_13 -> S11_12
- S13 pad DI: S11_13 -> S12_13
Routing:
- net S11_13: track 38.7 -> 0.00 mm, vias 2 -> 0
- net VCC: track 2422.4 -> 2456.9 mm, vias 16 -> 17
- net S11_12: track 0.00 -> 33.8 mm, vias 0 -> 2
- net S12_13: track 0.00 -> 29.1 mm, vias 0 -> 2
- net r5: track 556.4 -> 579.7 mm
- net c2: track 157.5 -> 178.4 mm
- net GND: track 2360.6 -> 2379.5 mm, vias 100 -> 101
- net r1: track 348.3 -> 366.8 mm
- net led1_11: track 61.9 -> 78.1 mm, vias 2 -> 3
- net c0: track 177.1 -> 192.1 mm, vias 2 -> 4
- net sclL: track 152.5 -> 137.4 mm
- net c1: track 184.7 -> 199.6 mm
- net sdaL: track 151.0 -> 136.3 mm
- net r4: track 491.7 -> 504.5 mm, vias 4 -> 6
- net encAR: track 122.2 -> 110.3 mm
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Other:
- outline, holes or cut-outs redrawn
- board text added: "anise90a/anise85a(v0.2) PCB designed by AniseHID/ngzh (evolved from GH60 by komar007 & jdcarpe)"
- board text removed: "anise90a/anise85a(v0.1) PCB designed by AniseHID/ngzh"
